File: Gimbal Board/GimbalMotorController2017.sch (EAGLE design)
At the start: 122 parts, among them J1 SL03THROUGH_HOLE, J3 APP_2POS_CONFIG5V_HORIZ, Q7 MOSFET-PCHANNEL, Q8 MOSFET-PCHANNEL, Q9 MOSFET-NCHANNELAO3404A, U1 NUP4201MR6, U2 MAX3232D, U3 CSD18533Q5A, U4 CSD18533Q5A, U5 CSD18533Q5A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

Commit message: Reorganized schematic sections
Added new section for MAX232 and reorganized External connections for clarity
Other:
- note added: "MAX232"
- moved on the sheet: C44, C45, C46, C47, C48, J3GND, J3VCC, U$2, U$5, U$6, U$7, U2
