File: _autosave-Gimbal-Powerboard.kicad_pcb (KiCad board)
At the start: 2 copper layers, 165 parts, among them Q1 Q_PMOS_GDS, Q2 Q_PMOS_GDS, Q3 SI4116DY, Q4 SI4116DY, Q5 SI4116DY, Q6 SI4116DY, Q7 SI4116DY, Q8 SI4116DY, U1 DRV8301, U2 NUP4201MR6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

Commit message: Sorted PCB components, preliminary layout
Parts:
- moved D16 350.5 mm to (317.6, 132.5)
- moved C32 349.8 mm to (357.3, 148.0)
- moved D12 348.0 mm to (318.6, 147.7)
- moved D14 345.1 mm to (335.4, 105.0)
- moved TP6 339.8 mm to (341.4, 138.4)
- moved R27 332.3 mm to (337.4, 144.3)
- moved D15 332.1 mm to (332.6, 75.6)
- moved R29 322.4 mm to (349.6, 151.0)
- moved TP9 314.7 mm to (346.1, 127.6)
- moved C7 313.4 mm to (342.3, 92.3)
- moved R33 310.1 mm to (347.9, 98.3)
- moved TP11 307.6 mm to (347.3, 84.6)
- moved TP3 304.3 mm to (332.6, 136.9)
- moved C11 301.7 mm to (348.7, 91.8)
- moved TP10 299.7 mm to (341.8, 41.4)
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