File: _saved_Gimbal-Powerboard.sch (KiCad schematic (older format))
At the start: 129 parts, among them Q1 Q_PMOS_GDS, Q2 Q_PMOS_GDS, Q3 SI4116DY, Q4 SI4116DY, Q5 SI4116DY, Q6 SI4116DY, Q7 SI4116DY, Q8 SI4116DY, U1 DRV8301, U2 NUP4201MR6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

Commit message: Sorted PCB components, preliminary layout
Parts:
- C37: symbol Anderson-2 -> Anderson_2
- U5: symbol Molex_SL-3 -> Molex_SL_3
- U6: symbol Molex_SL-5 -> Molex_SL_5
Other:
- moved on the sheet: C28, C35, C36, C37, C38, C39, C41, C42, C43, TP12, TP13, TP14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
