File: Gimbal-Powerboard.sch (KiCad schematic (older format))
At the start: 116 parts, among them Q1 Q_PMOS_GDS, Q2 Q_PMOS_GDS, Q3 R6020ENJSMD, Q4 R6020ENJSMD, Q5 R6020ENJSMD, Q6 R6020ENJSMD, Q7 R6020ENJSMD, Q8 R6020ENJSMD, U1 DRV8301, U2 NUP4201MR6, U3 LAUNCHXL-F28069M_Launchpad_J1, U4 MAX3232, U5 Molex_SL-3, U6 Molex_SL-5, U7 ACS711, U8 ACS711

Commit message: Changed MAX3232 device, updated GND and VCC flags, added 100k pull down resistor in parallel with zener diode, added diode across 10 ohm resistor for all phases, added flags for motor terminal A,B,C
Parts:
- removed U4: MAX3232, MRDT_ICs:SOIC_16_3.9x9.9mm_Pitch1.27mm, symbol MAX3232
- removed U8: ACS711, ACS711:SOIC127P600X175-8N, symbol ACS711
- added D12, D13, D14, D15, D16, D17: D, symbol D
- added R26, R27, R34, R35, R36: 100k, symbol R
- added R37: 1k, Resistors_SMD:R_0805_HandSoldering, symbol R
- added U4: ACS711, ACS711:SOIC127P600X175-8N, symbol ACS711
- added U8: MAX_3232, symbol MAX_3232
- C35, C36, C41, C42, C43: value 0.1u -> 1uF
- R16: value 1k -> 100k; footprint Resistors_SMD:R_0805_HandSoldering -> (none)
Connections:
- net SH_C is gone; now on net MTC: C21.2, C40.1, D9.2 (A), Q3.3 (S), Q6.1 (D), TP9.1, U1.36 (SH_C)
- net 232_RX: now also U8.13 (RIN1)
- net 232_TX: now also U8.14 (DOUT1)
- net CURRENTSENSEA: now also C27.1, U4.7 (VIOUT); no longer C11.1, U7.7 (VIOUT)
- net CURRENTSENSEB: now also C11.1, U7.7 (VIOUT); no longer C27.1
- net GH_A: now also D17.1 (K)
- net GH_B: now also D15.1 (K)
- net GH_C: now also D16.1 (K)
- net GL_A: now also D13.1 (K)
- net GL_B: now also D14.1 (K)
- net GL_C: now also D12.1 (K)
- net GND: now also C1.2, C2.2, C3.2, R16.2, R5.2, R27.2, R34.2, U4.5 (GND), U8.15 (GND)
- net SH_A: now also R35.2, U4.1 (IP+), U4.2 (IP+); no longer C38.1, R30.2
- net SH_B: now also R36.2; no longer C39.1
- net UART_RX: now also U8.12 (ROUT1)
- net UART_TX: now also U8.11 (DIN1)
- net VCC: now also U5.2, R37.2, U4.8 (VCC), U8.16 (VCC); no longer R16.2
- net at D10.1 (K), Q4.2 (G), R24.1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: now also D17.2 (A), R35.1
- net at D7.1 (K), Q7.2 (G), R21.1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: now also D13.2 (A), R34.1
- net at D11.1 (K), Q5.2 (G), R25.1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: now also D15.2 (A), R36.1
- net at D8.1 (K), Q8.2 (G), R22.1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: now also R16.1, D14.2 (A)
- net MTB: now reaches R32.2, U7.3 (IP-), U7.4 (IP-)
- net MTB: now also C39.1
- net at D9.1 (K), Q3.2 (G), R23.1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: now also D16.2 (A), R26.1
- net at D6.1 (K), Q6.2 (G), R20.1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: now also D12.2 (A), R27.1
- net MTC: now reaches R28.2
- net MTC: now also R26.2
- net at C36.1: now also U8.1 (C1+)
- net at C42.2: now also U8.2 (V+)
- net at C36.2: now also U8.3 (C1-)
- net at C41.1: now also U8.4 (C2+)
- net at C41.2: now also U8.5 (C2-)
- net at C43.2: now also U8.6 (V-)
- new net: R37.1, U4.6 (FAULT)
- new net MTA: C38.1, R30.2, U4.3 (IP-), U4.4 (IP-)
- no-connect marks 7 -> 26
Other:
- note removed: "Add current sensor"
- moved on the sheet: C30, C31, C35, C36, C41, C42, C43, D6, D7, D8, R25, TP10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

Commit message: Initial PCB layout with 2P2T switch for PWM, INL_C
Parts:
- removed C38, C39, C40: Anderson-1, MRDT_Connectors:Anderson_1_Horisontal, symbol Anderson-1
- added C28, C38, C39: Anderson_1, MRDT_Connectors:Anderson_1_Horisontal, symbol Anderson_1
- added U27: 2P2T_Switch, MRDT_Switches:2P2T_Switch_GrayHill_Series76, symbol 2P2T_Switch
- D12, D13, D14, D15, D16, D17: footprint (none) -> Diodes_SMD:D_SOD-123
- Q3, Q4, Q5, Q6, Q7, Q8: value R6020ENJSMD -> SI4116DY; footprint MRDT_Actives:Rohm_R6020ENJ_N_Channel_MOSFET -> MRDT_Actives:SO-8_N_Si4116dy_nChannelMOSFET
- R16, R26, R27, R34, R35, R36: footprint (none) -> Resistors_SMD:R_0805_HandSoldering
- U3: footprint MRDT_Shields:LAUNCHXL_F28069M_Launchpad_J1 -> MRDT_Shields:LAUNCHXL_F28069M_Launchpad_J1_BottomSMD
- U8: footprint (none) -> MRDT_ICs:SOIC_16_3.9x9.9mm_Pitch1.27mm
Connections:
- net GND: now also C30.1; no longer C30.2
- net INL_C: now also U27.C2 (In2); no longer U3.P_5 (J4_35)
- net MTA: now also C28.1
- net MTB: now also C38.1
- net MTC: now also C39.1
- net PVDD: now also C30.2; no longer C30.1
- net PWM_IN: now also U27.C1 (In1); no longer U3.DAC2 (J4_31)
- net INL_C/PWM_IN_2: now reaches U3.P_44 (J2_18)
- net INL_C/PWM_IN_2: now also U27.C1_1 (Out1a), U27.C2_2 (Out2b)
- new net INL_C/PWM_IN_1: U27.C1_2 (Out1b), U27.C2_1 (Out2a), U3.P_5 (J4_35)
- no-connect marks 26 -> 25
Other:
- note added: "(Arrow is the direction of Depression)"
- note added: "*PWM is in C1\n INL_C is in C2"
- note added: "C1"
- note added: "C2"
- note added: "J1-INL_C\nJ5-PWM"
- note added: "J1-PWM\nJ5-INL_C\n"
- note added: "J5-->\nJ1<--"

Commit message: Sorted PCB components, preliminary layout
Parts:
- C37: symbol Anderson-2 -> Anderson_2
- U3: symbol LAUNCHXL-F28069M_Launchpad_J1 -> LAUNCHXL_F28069M_Launchpad_J1
- U5: symbol Molex_SL-3 -> Molex_SL_3
- U6: symbol Molex_SL-5 -> Molex_SL_5
Other:
- moved on the sheet: C28, C35, C36, C37, C38, C39, C41, C42, C43, TP12, TP13, TP14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

Commit message: Created traces for MAX3232, part of DRV8301
Parts:
- C10, C11, C12, C13, C14, C15, C16, C17, C18, C20, C21, C23, C24, C25, C26, C27, C3, C32, C33, C34, C35, C36, C4, C41, C42, C43, C6, C7, C8, C9: footprint Capacitors_SMD:C_0805_HandSoldering -> Capacitors_SMD:C_0603_HandSoldering
- R1, R10, R11, R12, R13, R14, R15, R16, R17, R18, R19, R2, R20, R21, R22, R23, R24, R25, R26, R27, R28, R29, R3, R30, R31, R32, R33, R34, R35, R36, R37, R4, R5, R6, R7, R8, R9: footprint Resistors_SMD:R_0805_HandSoldering -> Capacitors_SMD:C_0603_HandSoldering
Connections:
- net PVDD renamed 12VACT
- net PVDDSENSE renamed 12VACTSENSE

Commit message: Added ground copper layer, silkscreen for serial, pwm, phase connections, removed test point for MTC. Finished round 1 board review with Judah, Andrew, Jacob
Parts:
- removed TP9: TEST, Wire_Pads:SolderWirePad_single_1mmDrill, symbol TEST
Connections:
- no-connect marks 25 -> 26
Changed lines of the file:
@@
 LIBS:MRDT_Silkscreens
 LIBS:MRDT_Switches
+LIBS:Gimbal-Powerboard-cache
 EELAYER 25 0
 EELAYER END
@@
 $EndComp
 $Comp
-L TEST TP10
-U 1 1 5A804188
-P 12900 3300
-F 0 "TP10" H 12900 3600 50  0000 C BNN
-F 1 "TEST" H 12900 3550 50  0000 C CNN
-F 2 "Wire_Pads:SolderWirePad_single_1mmDrill" H 12900 3300 50  0001 C CNN
-F 3 "" H 12900 3300 50  0001 C CNN
-	1    12900 3300
-	1    0    0    -1
-$EndComp
-$Comp
 L R R30
 U 1 1 5A804898
@@
 $EndComp
 $Comp
-L TEST TP11
-U 1 1 5A81938A
-P 12950 6500
-F 0 "TP11" H 12950 6800 50  0000 C BNN
-F 1 "TEST" H 12950 6750 50  0000 C CNN
-F 2 "Wire_Pads:SolderWirePad_single_1mmDrill" H 12950 6500 50  0001 C CNN
-F 3 "" H 12950 6500 50  0001 C CNN
-	1    12950 6500
-	1    0    0    -1
-$EndComp
-$Comp
 L R R32
 U 1 1 5A819390
@@
 F 3 "" H 12450 10100 50  0001 C CNN
 	1    12450 10100
-	1    0    0    -1
-$EndComp
-$Comp
-L TEST TP9
-U 1 1 5A8382F0
-P 12900 9700
-F 0 "TP9" H 12900 10000 50  0000 C BNN
-F 1 "TEST" H 12900 9950 50  0000 C CNN
-F 2 "Wire_Pads:SolderWirePad_single_1mmDrill" H 12900 9700 50  0001 C CNN
-F 3 "" H 12900 9700 50  0001 C CNN
-	1    12900 9700
 	1    0    0    -1
 $EndComp
@@
 Wire Wire Line
 	13250 10250 13250 10500
-Connection ~ 12900 9750
-Wire Wire Line
-	12900 9700 12900 9750
 Connection ~ 12550 9650
 Wire Wire Line
@@
 Wire Wire Line
 	13350 7050 13350 7300
-Connection ~ 12950 6550
-Wire Wire Line
-	12950 6500 12950 6550
 Connection ~ 12600 6450
 Wire Wire Line
@@
 Connection ~ 13100 6550
 Wire Wire Line
-	13100 6550 12750 6550
-Wire Wire Line
-	13100 6150 13100 6550
+	12750 6550 13100 6550
+Wire Wire Line
+	13100 6550 13100 6150
 Wire Wire Line
 	13100 6150 13300 6150
@@
 Wire Wire Line
 	13150 3350 13350 3350
-Wire Wire Line
-	12900 3300 12900 3350
-Connection ~ 12900 3350
 Wire Wire Line
 	13650 3500 13350 3500
@@
 Wire Wire Line
 	19600 3100 19450 3100
+NoConn ~ 16100 3900
+Wire Wire Line
+	12900 3300 12900 3350
+Connection ~ 12900 3350
+$Comp
+L TEST TP10
+U 1 1 5A804188
+P 12900 3300
+F 0 "TP10" H 12900 3600 50  0000 C BNN
+F 1 "TEST" H 12900 3550 50  0000 C CNN
+F 2 "Wire_Pads:SolderWirePad_single_1mmDrill" H 12900 3300 50  0001 C CNN
+F 3 "" H 12900 3300 50  0001 C CNN
+	1    12900 3300
+	1    0    0    -1
+$EndComp
+Connection ~ 12950 6550
+Wire Wire Line
+	12950 6500 12950 6550
+$Comp
+L TEST TP11
+U 1 1 5A81938A
+P 12950 6500
+F 0 "TP11" H 12950 6800 50  0000 C BNN
+F 1 "TEST" H 12950 6750 50  0000 C CNN
+F 2 "Wire_Pads:SolderWirePad_single_1mmDrill" H 12950 6500 50  0001 C CNN
+F 3 "" H 12950 6500 50  0001 C CNN
+	1    12950 6500
+	1    0    0    -1
+$EndComp
 $EndSCHEMATC

Commit message: Updated flags to be directional
Connections:
- net 12VACT: no longer Q4.1 (D), Q5.1 (D)
- net GND: now also Q4.1 (D), Q5.1 (D)
Other:
- moved on the sheet: C30, C31, TP12, TP14, TP15

Commit message: Generated gerbs
Parts:
- C32, C33, C34: value 0.1u -> 0.01u
Connections:
- net 12VACT: now also Q4.1 (D), Q5.1 (D)
- net GND: no longer Q4.1 (D), Q5.1 (D)
- net DE: no longer names the net of U3.P_13 (J4_34)
- no-connect marks 26 -> 27
Other:
- moved on the sheet: C30
Changed lines of the file:
@@
 L C C30
 U 1 1 5A800D77
-P 13350 2300
-F 0 "C30" H 13375 2400 50  0000 L CNN
-F 1 "2.2u" H 13375 2200 50  0000 L CNN
-F 2 "Capacitors_SMD:C_1206_HandSoldering" H 13388 2150 50  0001 C CNN
-F 3 "" H 13350 2300 50  0001 C CNN
-	1    13350 2300
+P 13350 2450
+F 0 "C30" H 13375 2550 50  0000 L CNN
+F 1 "2.2u" H 13375 2350 50  0000 L CNN
+F 2 "Capacitors_SMD:C_1206_HandSoldering" H 13388 2300 50  0001 C CNN
+F 3 "" H 13350 2450 50  0001 C CNN
+	1    13350 2450
 	-1   0    0    1
 $EndComp
@@
 P 13800 4250
 F 0 "C33" H 13825 4350 50  0000 L CNN
-F 1 "0.1u" H 13825 4150 50  0000 L CNN
+F 1 "0.01u" H 13825 4150 50  0000 L CNN
 F 2 "Capacitors_SMD:C_0603_HandSoldering" H 13838 4100 50  0001 C CNN
 F 3 "" H 13800 4250 50  0001 C CNN
@@
 P 13800 7450
 F 0 "C34" H 13825 7550 50  0000 L CNN
-F 1 "0.1u" H 13825 7350 50  0000 L CNN
+F 1 "0.01u" H 13825 7350 50  0000 L CNN
 F 2 "Capacitors_SMD:C_0603_HandSoldering" H 13838 7300 50  0001 C CNN
 F 3 "" H 13800 7450 50  0001 C CNN
@@
 P 13700 10650
 F 0 "C32" H 13725 10750 50  0000 L CNN
-F 1 "0.1u" H 13725 10550 50  0000 L CNN
+F 1 "0.01u" H 13725 10550 50  0000 L CNN
 F 2 "Capacitors_SMD:C_0603_HandSoldering" H 13738 10500 50  0001 C CNN
 F 3 "" H 13700 10650 50  0001 C CNN
@@
 Text GLabel 15950 3500 0    49   BiDi ~ 0
 INL_C/PWM_IN_1
-Text GLabel 15950 3600 0    49   Input ~ 0
-DE
 Text GLabel 19600 3600 2    49   Input ~ 0
 CURRENTSENSEA
@@
 Text GLabel 14400 3550 3    49   UnSpc ~ 0
 GND
-Text GLabel 13750 2550 3    49   UnSpc ~ 0
+Text GLabel 14050 2500 3    49   UnSpc ~ 0
 GND
 Text GLabel 18400 2900 1    49   Input ~ 0
@@
 	1    0    0    -1
 $EndComp
-Text GLabel 13750 5750 3    49   UnSpc ~ 0
+Text GLabel 13350 5650 3    49   UnSpc ~ 0
 GND
 Wire Wire Line
@@
 	15950 3500 16100 3500
 Wire Wire Line
-	15950 3600 16100 3600
-Wire Wire Line
 	19450 3600 19600 3600
 Wire Wire Line
@@
 Wire Wire Line
 	14600 3050 14600 3100
-Wire Wire Line
-	12550 2450 14550 2450
 Wire Wire Line
 	14550 2750 14550 3150
@@
 Connection ~ 14400 3450
 Wire Wire Line
-	12550 2450 12550 2600
-Wire Wire Line
-	13750 2450 13750 2550
-Connection ~ 13350 2450
-Connection ~ 13750 2450
-Wire Wire Line
-	13350 2150 13350 2100
+	12550 2300 12550 2600
 Wire Wire Line
 	13350 2100 13400 2100
@@
 Connection ~ 14450 6700
 Wire Wire Line
-	12550 5650 14600 5650
-Wire Wire Line
-	13750 5650 13750 5750
-Wire Wire Line
 	13400 5300 13350 5300
 Wire Wire Line
 	13350 5300 13350 5350
-Connection ~ 13750 5650
-Wire Wire Line
-	12550 5650 12550 5800
-Connection ~ 13350 5650
+Wire Wire Line
+	12550 5350 12550 5800
 Wire Wire Line
 	12550 6600 12600 6600
@@
 Wire Wire Line
 	18000 4850 18350 4850
+Wire Wire Line
+	13350 2100 13350 2300
+Wire Wire Line
+	13350 2300 12550 2300
+Text GLabel 13350 2600 3    49   UnSpc ~ 0
+GND
+Wire Wire Line
+	14550 2450 14550 2400
+Wire Wire Line
+	14550 2400 14050 2400
+Wire Wire Line
+	14050 2400 14050 2500
+Wire Wire Line
+	13350 5350 12550 5350
+Text GLabel 14200 5650 3    49   UnSpc ~ 0
+GND
+Wire Wire Line
+	14600 5650 14600 5550
+Wire Wire Line
+	14600 5550 14200 5550
+Wire Wire Line
+	14200 5550 14200 5650
+NoConn ~ 16100 3600
 $EndSCHEMATC
