File: Gimbal-Powerboard.kicad_pcb (KiCad board)
At the start: 2 copper layers, 59.7 x 124.9 mm, 170 parts, among them Q1 Q_PMOS_GDS, Q2 Q_PMOS_GDS, Q3 SI4116DY, Q4 SI4116DY, Q5 SI4116DY, Q6 SI4116DY, Q7 SI4116DY, Q8 SI4116DY, U1 DRV8301, U2 NUP4201MR6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

Commit message: Fixed an issue with drill holes not rendering properly in gerb viewers. Generated fixed gerbs and updated the zip file
Parts:
- moved U5 0.28 mm to (167.0, 39.6)
Routing:
- net GND: track 359.2 -> 343.6 mm
Changed lines of the file:
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@@
     (thickness 1.6)
     (drawings 48)
-    (tracks 1656)
+    (tracks 1654)
     (zones 0)
     (modules 170)
@@
     (35 F.Paste user)
     (36 B.SilkS user)
-    (37 F.SilkS user hide)
+    (37 F.SilkS user)
     (38 B.Mask user)
     (39 F.Mask user)
@@
     (pad_to_mask_clearance 0.2)
     (aux_axis_origin 0 0)
-    (visible_elements 7FFFFDFF)
+    (visible_elements 7FFCFFFF)
     (pcbplotparams
       (layerselection 0x010f0_80000001)
@@
   )
   (module MRDT_Connectors:MOLEX_SL_3_Horizontal (layer F.Cu)
-    (at 167.259 39.751)
+    (at 167.005 39.624)
     (fp_text reference U5 (at -1.27 2.54) (layer F.SilkS) hide
       (effects (font (size 1 1) (thickness 0.15)))
@@
   (segment (start 152.052 84.709) (end 153.736 84.709) (width 0.254) (layer B.Cu) (net 1))
   (segment (start 153.736 84.709) (end 153.797 84.648) (width 0.254) (layer B.Cu) (net 1))
-  (segment (start 169.799 39.751) (end 169.799 41.5925) (width 0.254) (layer F.Cu) (net 1))
-  (segment (start 166.7891 44.6024) (end 157.352 44.6024) (width 0.254) (layer F.Cu) (net 1))
-  (segment (start 169.799 41.5925) (end 166.7891 44.6024) (width 0.254) (layer F.Cu) (net 1))
   (segment (start 143.952 50.546) (end 143.952 49.8475) (width 0.254) (layer B.Cu) (net 1))
   (segment (start 143.952 49.8475) (end 143.952 49.845) (width 0.254) (layer B.Cu) (net 1))
@@
   (segment (start 127.188 92.3848) (end 126.9746 92.5982) (width 0.254) (layer F.Cu) (net 4))
   (segment (start 126.9492 92.5728) (end 126.9746 92.5982) (width 0.25) (layer F.Cu) (net 4))
+  (segment (start 165.227 41.402) (end 165.227 41.91) (width 0.25) (layer B.Cu) (net 5))
+  (segment (start 165.227 99.06) (end 164.465 99.822) (width 0.254) (layer B.Cu) (net 5))
+  (segment (start 164.465 99.822) (end 164.465 100.203) (width 0.254) (layer B.Cu) (net 5))
+  (via (at 164.465 100.203) (size 0.6) (drill 0.4) (layers F.Cu B.Cu) (net 5))
+  (segment (start 163.068 100.203) (end 164.465 100.203) (width 0.254) (layer F.Cu) (net 5))
+  (segment (start 165.227 41.91) (end 165.227 45.339) (width 0.254) (layer B.Cu) (net 5))
+  (segment (start 165.227 45.339) (end 165.227 99.06) (width 0.254) (layer B.Cu) (net 5))
+  (segment (start 165.227 41.402) (end 167.005 39.624) (width 0.25) (layer B.Cu) (net 5))
   (segment (start 148.717 88.392) (end 148.5265 88.392) (width 0.254) (layer F.Cu) (net 5))
   (segment (start 148.717 88.392) (end 151.892 88.392) (width 0.254) (layer F.Cu) (net 5))
@@
   (segment (start 148.5265 88.392) (end 148.336 88.2015) (width 0.254) (layer B.Cu) (net 5))
   (via (at 148.5265 88.392) (size 0.6) (drill 0.4) (layers F.Cu B.Cu) (net 5))
-  (segment (start 165.227 45.339) (end 165.227 99.06) (width 0.254) (layer B.Cu) (net 5))
-  (segment (start 165.227 41.91) (end 165.227 45.339) (width 0.254) (layer B.Cu) (net 5))
-  (segment (start 167.259 39.878) (end 165.227 41.91) (width 0.254) (layer B.Cu) (net 5))
-  (segment (start 164.465 100.203) (end 163.068 100.203) (width 0.254) (layer F.Cu) (net 5))
-  (via (at 164.465 100.203) (size 0.6) (drill 0.4) (layers F.Cu B.Cu) (net 5))
-  (segment (start 164.465 99.822) (end 164.465 100.203) (width 0.254) (layer B.Cu) (net 5))
-  (segment (start 165.227 99.06) (end 164.465 99.822) (width 0.254) (layer B.Cu) (net 5))
-  (segment (start 167.259 39.751) (end 167.259 39.878) (width 0.254) (layer B.Cu) (net 5))
   (segment (start 145.669 54.798) (end 145.669 56.007) (width 0.254) (layer B.Cu) (net 5))
   (segment (start 145.669 56.007) (end 145.669 55.9308) (width 0.254) (layer B.Cu) (net 5))
@@
   (segment (start 136.398 55.8165) (end 136.2075 56.007) (width 0.254) (layer B.Cu) (net 5))
   (segment (start 135.001 54.798) (end 136.398 54.798) (width 0.254) (layer B.Cu) (net 5))
-  (segment (start 167.259 39.751) (end 167.005 39.751) (width 0.254) (layer B.Cu) (net 5))
   (segment (start 145.381 99.248) (end 145.034 98.901) (width 0.254) (layer F.Cu) (net 5))
   (segment (start 157.226 97.5868) (end 157.226 99.1235) (width 0.254) (layer F.Cu) (net 5))
@@
   (segment (start 133.353388 106.937388) (end 135.258388 106.937388) (width 0.254) (layer F.Cu) (net 71))
   (segment (start 132.807392 106.391392) (end 133.353388 106.937388) (width 0.254) (layer F.Cu) (net 71))
+  (segment (start 164.465 39.624) (end 164.465 96.901) (width 0.25) (layer B.Cu) (net 84))
   (segment (start 158.242 117.094) (end 136.906 117.094) (width 0.254) (layer F.Cu) (net 84))
   (segment (start 136.906 117.094) (end 136.144 117.094) (width 0.254) (layer F.Cu) (net 84))
@@
   (segment (start 136.144 117.094) (end 135.382 116.332) (width 0.254) (layer F.Cu) (net 84))
   (segment (start 135.382 116.332) (end 128.905 116.332) (width 0.254) (layer F.Cu) (net 84))
-  (segment (start 127.635 115.062) (end 128.905 116.332) (width 0.254) (layer F.Cu) (net 84))
+  (segment (start 128.905 116.332) (end 127.635 115.062) (width 0.254) (layer F.Cu) (net 84))
   (segment (start 158.242 117.094) (end 161.6075 117.094) (width 0.254) (layer F.Cu) (net 84))
   (segment (start 164.719 98.8568) (end 163.703 99.8728) (width 0.254) (layer B.Cu) (net 84))
   (segment (start 163.703 99.8728) (end 163.703 114.1984) (width 0.254) (layer B.Cu) (net 84))
-  (segment (start 164.719 98.8568) (end 164.719 39.751) (width 0.254) (layer B.Cu) (net 84))
   (segment (start 163.703 114.9985) (end 161.6075 117.094) (width 0.254) (layer B.Cu) (net 84))
+  (segment (start 164.719 97.155) (end 164.719 98.8568) (width 0.25) (layer B.Cu) (net 84))
+  (segment (start 164.465 96.901) (end 164.719 97.155) (width 0.25) (layer B.Cu) (net 84))
   (segment (start 150.8125 86.487) (end 151.1935 86.868) (width 0.254) (layer B.Cu) (net 87))
   (segment (start 147.1168 87.8332) (end 147.193 87.757) (width 0.254) (layer B.Cu) (net 87))

Commit message: Made some last minute adjustments to the silkscreen for clarity
Other:
- board text added: "GND"
Changed lines of the file:
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@@
     (links 340)
     (no_connects 2)
-    (area 103.673 16.107999 202.149255 151.7436)
+    (area 113.208999 26.404499 173.049001 151.459001)
     (thickness 1.6)
-    (drawings 48)
+    (drawings 50)
     (tracks 1654)
     (zones 0)
@@
   (page A4)
   (layers
-    (0 F.Cu signal)
-    (31 B.Cu signal)
+    (0 F.Cu signal hide)
+    (31 B.Cu signal hide)
     (32 B.Adhes user)
     (33 F.Adhes user)
@@
     (35 F.Paste user)
     (36 B.SilkS user)
-    (37 F.SilkS user)
+    (37 F.SilkS user hide)
     (38 B.Mask user)
     (39 F.Mask user)
@@
     (pad_to_mask_clearance 0.2)
     (aux_axis_origin 0 0)
-    (visible_elements 7FFCFFFF)
+    (visible_elements 7FFEFF7F)
     (pcbplotparams
       (layerselection 0x010f0_80000001)
@@
     (tags SOD-323)
     (attr smd)
-    (fp_text reference D5 (at 0 -1.524 90) (layer F.SilkS)
+    (fp_text reference D5 (at 0.127 -1.524 90) (layer F.SilkS)
       (effects (font (size 1 1) (thickness 0.15)))
     )
@@
       (effects (font (size 1 1) (thickness 0.15)))
     )
-    (fp_text value 33u (at -2.54 -5.08 90) (layer F.SilkS)
+    (fp_text value 33u (at -4.699 -2.286 180) (layer F.SilkS) hide
       (effects (font (size 1 1) (thickness 0.15)))
     )
@@
     (tags "capacitor 0603")
     (attr smd)
-    (fp_text reference C12 (at 0.0508 1.3208 90) (layer F.SilkS)
+    (fp_text reference C12 (at 3.175 0 90) (layer F.SilkS)
       (effects (font (size 1 1) (thickness 0.15)))
     )
@@
     (tags "capacitor 0603")
     (attr smd)
-    (fp_text reference C15 (at 0 -1.25 90) (layer F.SilkS)
+    (fp_text reference C15 (at -3.175 0.127 90) (layer F.SilkS)
       (effects (font (size 1 1) (thickness 0.15)))
     )
@@
     (tags "capacitor 0603")
     (attr smd)
-    (fp_text reference C16 (at 0.1016 -1.1684 90) (layer F.SilkS)
+    (fp_text reference C16 (at 3.2766 -0.0254 90) (layer F.SilkS)
       (effects (font (size 1 1) (thickness 0.15)))
     )
@@
     (tags "capacitor 0603")
     (attr smd)
-    (fp_text reference C23 (at 3.175 0 90) (layer F.SilkS)
+    (fp_text reference C23 (at 0.0635 -1.143 90) (layer F.SilkS)
       (effects (font (size 1 1) (thickness 0.15)))
     )
@@
     (tags "capacitor 0603")
     (attr smd)
-    (fp_text reference C24 (at 3.175 0 90) (layer F.SilkS)
+    (fp_text reference C24 (at -0.127 -1.27 90) (layer F.SilkS)
       (effects (font (size 1 1) (thickness 0.15)))
     )
@@
     (tags "capacitor 0603")
     (attr smd)
-    (fp_text reference R4 (at 0 -1.25 270) (layer F.SilkS)
+    (fp_text reference R4 (at 0 1.27 270) (layer F.SilkS)
       (effects (font (size 1 1) (thickness 0.15)))
     )
@@
       (xy 10.42777 15.665413) (xy 10.448357 15.679839) (xy 10.468725 15.683261) (xy 10.490644 15.648548)) (layer B.SilkS) (width 0.01))
   )
+  (gr_text GND (at 161.417 44.45 270) (layer F.SilkS)
+    (effects (font (size 1 1) (thickness 0.25)))
+  )
+  (gr_text 12VACT (at 145.669 44.577 90) (layer F.SilkS)
+    (effects (font (size 1 1) (thickness 0.25)))
+  )
   (gr_text C (at 120.777 42.418) (layer F.SilkS)
